File: hardware/lcd.kicad_sch (KiCad schematic)
At the start: 8 parts, among them J2 AYF531035, U6 SN74LV4T125, U7 SN74LV1T34

Commit message: LCD sheet: move U6 to the 3.5x3.5 mm RGY package
SN74LV4T125RGYR replaces the TSSOP-14 part to save board area. The
project footprint follows TI's RGY0014A land pattern (4219040/A):
0.24 x 0.6 mm pads at 0.5 mm pitch, 2.05 mm exposed pad (pin 15, tied
to GND through a hidden symbol pin) with a 2x2 paste split.
ERC is clean with all severities enabled.

Co-Authored-By: Claude Opus 5.5 (1M context) <noreply@anthropic.com>
Parts:
- U6: footprint Package_SO:TSSOP-14_4.4x5mm_P0.65mm -> Eigentime32:Texas_RGY0014A_VQFN-14-1EP_3.5x3.5mm_P0.5mm_EP2.05x2.05mm; MPN SN74LV4T125PWR -> SN74LV4T125RGYR
Connections:
- net GND: now also U6.15 (GND)
Changed lines of the file:
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@@
 		(property "Reference" "U6" (at 119.38 106.68 0) (effects (font (size 1.27 1.27)) (justify left)))
 		(property "Value" "SN74LV4T125" (at 119.38 109.22 0) (effects (font (size 1.27 1.27)) (justify left)))
-		(property "Footprint" "Package_SO:TSSOP-14_4.4x5mm_P0.65mm" (at 127 88.9 0) (effects (font (size 1.27 1.27)) (hide yes)))
+		(property "Footprint" "Eigentime32:Texas_RGY0014A_VQFN-14-1EP_3.5x3.5mm_P0.5mm_EP2.05x2.05mm" (at 127 88.9 0) (effects (font (size 1.27 1.27)) (hide yes)))
 		(property "Datasheet" "https://www.ti.com/lit/ds/symlink/sn74lv4t125.pdf" (at 127 88.9 0) (effects (font (size 1.27 1.27)) (hide yes)))
 		(property "Description" "LCD SCLK/SI/SCS/DISP buffer on VLCD; Ioff 5 uA max" (at 127 88.9 0) (effects (font (size 1.27 1.27)) (hide yes)))
 		(property "Manufacturer" "Texas Instruments" (at 127 88.9 0) (effects (font (size 1.27 1.27)) (hide yes)))
-		(property "MPN" "SN74LV4T125PWR" (at 127 88.9 0) (effects (font (size 1.27 1.27)) (hide yes)))
+		(property "MPN" "SN74LV4T125RGYR" (at 127 88.9 0) (effects (font (size 1.27 1.27)) (hide yes)))
 		(pin "1")
 		(pin "10")
@@
 		(pin "13")
 		(pin "14")
+		(pin "15")
 		(pin "2")
 		(pin "3")
