File: hardware/Eigentime32.kicad_sch (KiCad schematic)
At the start: 0 parts

Commit message: Full schematic: power, RTC, MCU, LCD and NFC sheets (#2)
* Add Power schematic sheet

CR2032 in a Keystone 3034 SMT retainer, DMG2305UX P-FET reverse
protection (gate to GND), 100 uF + 100 nF on VBAT, and a TPS61099
adjustable boost set to 3.0 V (R1 402k / R2 200k, 1 uH WE-LQS,
10 uF CIN, 2 x 10 uF COUT, 1M pull-down on EN). The sheet exposes
VBAT, VLCD and LCD_PWR_EN as hierarchical pins. ERC is clean with
all severities enabled.

Co-Authored-By: Claude Opus 5.5 (1M context) <noreply@anthropic.com>

* Power sheet: add TPS22916C switch ahead of the LCD boost

U5 (TPS22916CYFPR) on LCD_PWR_EN cuts the TPS61099's 0.5-1.6 uA
shutdown current and the 100 uF bulk's leakage off the cell while the
lid is shut. C2 moves to the switched boost input behind R4 (470R),
which limits inrush to ~6.6 mA; the switch's own slew would draw
220-350 mA. R5/C8 (1M/470n) delay the boost EN until C2 has charged.
Always-on VBAT keeps 100 nF + 1 uF.

Adds a project symbol library with the TPS22916C symbol; the footprint
is the TI PicoStar 2x2 0.4 mm land pattern, which matches YFP.
ERC is clean with all severities enabled.

Co-Authored-By: Claude Opus 5.5 (1M context) <noreply@anthropic.com>

* Add RTC schematic sheet

RV-3032-C7 (project symbol, RV-3032 pinout) on always-on VBAT with
100 nF decoupling, 10k I2C pull-ups, 470k INT pull-up, EVI tied high
and a CLKOUT test pad. VBAT, SDA, SCL, RTC_INT and RTC_CLKOUT are
hierarchical pins.

No VBACKUP bridge: the pin is tied to VSS through 10k with switchover
off (BSM = 00). An MLCC's IR spec (50 MOhm.uF, i.e. a 50 s
self-discharge time constant) can't guarantee a 60 s cell swap at any
size, and its worst-case leakage would exceed the ~1 uA budget. C1 is
removed from the BOM. ERC is clean with all severities enabled.

Co-Authored-By: Claude Opus 5.5 (1M context) <noreply@anthropic.com>

* Add MCU sheet and update design docs

STM32L031G6U6 (UFQFPN28) on VBAT with ST's decoupling (10 uF bulk
fitted as DNP because of IR leakage), NRST filter, BOOT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
Other:
- added sheet LCD (lcd.kicad_sch)
- added sheet MCU (mcu.kicad_sch)
- added sheet NFC (nfc.kicad_sch)
- added sheet Power (power.kicad_sch)
- added sheet RTC (rtc.kicad_sch)
