File: hardware/nfc.kicad_sch (KiCad schematic)
At the start: 6 parts, among them U8 ST25DV04KC-IE6C3

Commit message: Layout phase 1: placement, NFC coil, part picks for TBD footprints
Board: 40 mm round, 0.8 mm, 2 layers. Front carries only the NFC coil
(LCD keep-out rule area); every other part is on the back around the
centred CR2032 holder (nothing taller than its 4.06 mm). Buttons at
12 o'clock, hinge mark at 9, lid sensor at 3, LCD FPC connector at 6.
Rules: 0.15 mm clearance, 0.2 mm tracks, 0.5/0.3 mm vias, 0.3 mm
copper-to-edge. A rule area forbids copper pour anywhere inside the
coil. Reference designators are on the fab layers.

NFC coil: 8-turn Archimedean spiral on F.Cu, 38.1 mm OD, 0.15/0.15 mm,
built as one polygon in a net-tie footprint (AE1) with plated terminal
vias at 4-5 o'clock next to U8.

Parts: lid sensor is now an Allegro CT8132SK-IS3 TMR switch (push-pull,
no pull-up; SMD NC reeds don't fit and the Coto RR122 is obsolete);
buttons are Panasonic EVQ-P7A01P side-push switches. MCU sheet, BOM
and docs updated. KiCad-written project defaults in .kicad_pro are
included.

ERC clean; DRC: 0 violations, 0 parity issues, only unrouted nets.
Renders in docs/renders.

Co-Authored-By: Claude Opus 5.5 (1M context) <noreply@anthropic.com>
Parts:
- AE1: footprint Eigentime32:NFC_PCB_Coil_D39mm_Placeholder -> Eigentime32:NFC_PCB_Coil_D38.1mm_8T; now left out of the parts list
Changed lines of the file:
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@@
 	)
 	(symbol (lib_id "Device:Antenna_Loop") (at 165.1 86.36 0) (unit 1)
-		(exclude_from_sim no) (in_bom yes) (on_board yes) (dnp no)
+		(exclude_from_sim no) (in_bom no) (on_board yes) (dnp no)
 		(property "Reference" "AE1" (at 170.18 81.28 0) (effects (font (size 1.27 1.27)) (justify left)))
 		(property "Value" "NFC coil" (at 170.18 83.82 0) (effects (font (size 1.27 1.27)) (justify left)))
-		(property "Footprint" "Eigentime32:NFC_PCB_Coil_D39mm_Placeholder" (at 165.1 86.36 0) (effects (font (size 1.27 1.27)) (hide yes)))
+		(property "Footprint" "Eigentime32:NFC_PCB_Coil_D38.1mm_8T" (at 165.1 86.36 0) (effects (font (size 1.27 1.27)) (hide yes)))
 		(property "Datasheet" "~" (at 165.1 86.36 0) (effects (font (size 1.27 1.27)) (hide yes)))
 		(property "Description" "PCB loop, target ~4.8 uH with the 28.5 pF internal tuning cap; drawn in layout" (at 165.1 86.36 0) (effects (font (size 1.27 1.27)) (hide yes)))
