File: hardware/mcu.kicad_sch (KiCad schematic)
At the start: 15 parts, among them J1 TC2030-NL, SW1 Reed (NC), SW2 BTN1, SW3 BTN2, U2 STM32L031G6U6

Commit message: Layout phase 1: placement, NFC coil, part picks for TBD footprints
Board: 40 mm round, 0.8 mm, 2 layers. Front carries only the NFC coil
(LCD keep-out rule area); every other part is on the back around the
centred CR2032 holder (nothing taller than its 4.06 mm). Buttons at
12 o'clock, hinge mark at 9, lid sensor at 3, LCD FPC connector at 6.
Rules: 0.15 mm clearance, 0.2 mm tracks, 0.5/0.3 mm vias, 0.3 mm
copper-to-edge. A rule area forbids copper pour anywhere inside the
coil. Reference designators are on the fab layers.

NFC coil: 8-turn Archimedean spiral on F.Cu, 38.1 mm OD, 0.15/0.15 mm,
built as one polygon in a net-tie footprint (AE1) with plated terminal
vias at 4-5 o'clock next to U8.

Parts: lid sensor is now an Allegro CT8132SK-IS3 TMR switch (push-pull,
no pull-up; SMD NC reeds don't fit and the Coto RR122 is obsolete);
buttons are Panasonic EVQ-P7A01P side-push switches. MCU sheet, BOM
and docs updated. KiCad-written project defaults in .kicad_pro are
included.

ERC clean; DRC: 0 violations, 0 parity issues, only unrouted nets.
Renders in docs/renders.

Co-Authored-By: Claude Opus 5.5 (1M context) <noreply@anthropic.com>
Parts:
- removed R11: 1M, Resistor_SMD:R_0402_1005Metric, symbol Device:R_Small
- removed SW1: Reed (NC), symbol Switch:SW_Reed_Opener
- added C23: 1u, Capacitor_SMD:C_0402_1005Metric, symbol Device:C_Small
- added U9: CT8132SK-IS3, Package_TO_SOT_SMD:SOT-23, symbol Eigentime32:CT8132SK-IS3
- J1: now left out of the parts list
- SW2, SW3: footprint (none) -> Button_Switch_SMD:SW_SPST_EVQP7A; MPN (none) -> EVQ-P7A01P; Manufacturer (none) -> Panasonic
Connections:
- net GND: now also C23.2, U9.3 (GND)
- net VBAT: now also C23.1, U9.1 (VDD)
- net LID_N renamed LID_CLOSED_N
- net LID_CLOSED_N: now also U9.2 (~{OUT})
Other:
- note added: "Wake sources use distinct EXTI lines: RTC_INT PA0 (EXTI0, WKUP1), BTN2 PB1 (EXTI1), LID PA2 (EXTI2, WKUP3), BTN1 PA3 (EXTI3), NFC_GPO PA8 (EXTI8). Any EXTI line wakes Stop mode. LCD: SPI1 SCK PA5 / MOSI PA7 (AF0); SCS PA4 and DISP PA6 as GPIO. I2C1 PB6/PB7 (AF1). Spares (no-connect): PA9/PA10 (USART2 TX/RX for a debug UART), PA15, PB3, PC14, PC15. Lid: CT8132 push-pull, low while the lid is shut;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"
- note removed: "Wake sources use distinct EXTI lines: RTC_INT PA0 (EXTI0, WKUP1), BTN2 PB1 (EXTI1), LID PA2 (EXTI2, WKUP3), BTN1 PA3 (EXTI3), NFC_GPO PA8 (EXTI8). Any EXTI line wakes Stop mode. LCD: SPI1 SCK PA5 / MOSI PA7 (AF0); SCS PA4 and DISP PA6 as GPIO. I2C1 PB6/PB7 (AF1). Spares (no-connect): PA9/PA10 (USART2 TX/RX for a debug UART), PA15, PB3, PC14, PC15. Pull-ups: internal pull-ups off on LID/BTN pins; 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"

Commit message: Layout: re-place parts around the CR2032 insertion channel
The Keystone 3034 is a tunnel retainer: the cell slides in flat from
12 o'clock with ~0.5 mm headroom, so a 21 mm wide path from the holder
to the board edge must be free of parts. A back-side rule area now
keeps it clear. The MCU, RTC and buttons moved out of it: MCU and RTC
on the right, buttons at ~10 and ~2 o'clock, lid sensor at ~4, SWD
pads at ~7:30, power on the left.

The TC2030 footprint is a project copy whose small via keep-out allows
nearby footprints (KiCad checks footprint keep-outs against bounding
boxes, and the holder's box covered it).

DRC: 0 violations, 0 parity issues; nets still unrouted.

Co-Authored-By: Claude Opus 5.5 (1M context) <noreply@anthropic.com>
Parts:
- J1: footprint Connector:Tag-Connect_TC2030-IDC-NL_2x03_P1.27mm_Vertical -> Eigentime32:Tag-Connect_TC2030-IDC-NL_2x03_P1.27mm_Vertical_FootprintsAllowed
Changed lines of the file:
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@@
 		(property "Reference" "J1" (at 48.26 99.06 0) (effects (font (size 1.27 1.27)) (justify left)))
 		(property "Value" "TC2030-NL" (at 48.26 101.6 0) (effects (font (size 1.27 1.27)) (justify left)))
-		(property "Footprint" "Connector:Tag-Connect_TC2030-IDC-NL_2x03_P1.27mm_Vertical" (at 60.96 101.6 0) (effects (font (size 1.27 1.27)) (hide yes)))
+		(property "Footprint" "Eigentime32:Tag-Connect_TC2030-IDC-NL_2x03_P1.27mm_Vertical_FootprintsAllowed" (at 60.96 101.6 0) (effects (font (size 1.27 1.27)) (hide yes)))
 		(property "Datasheet" "~" (at 60.96 101.6 0) (effects (font (size 1.27 1.27)) (hide yes)))
 		(property "Description" "SWD pads, no-legs footprint" (at 60.96 101.6 0) (effects (font (size 1.27 1.27)) (hide yes)))

Commit message: Layout-4l: fully routed 4-layer board, LCD FPC folds under the glass
- JLC04081H-3313 stackup (0.8 mm, 4 layers), In1/In2 signal, no pours;
  coil-ring keep-out on F/In1/In2. 0.45/0.3 mm vias (JLC free tier).
- Routed: 0 unrouted, DRC clean (all severities), schematic parity clean.
  75 vias, ~930 mm of track; 0.2 mm signal / 0.25 mm power, 37 short
  necks at 0.15-0.19 mm between pads.
- LCD FPC folds 180 deg under the glass (Sharp LD-26X06A Fig. 8-2) into
  J2 on the front at 180 deg, pad row y=+7.55, Panasonic land pattern
  (pad 1 = SCLK at +X). Panel on a 1.2 mm frame. LCD buffers, pull-ups
  and NFC VCC decoupling moved to the front under the panel, over the
  cell area where vias are free.
- Boost cluster hand-placed and locked: single short SW track, output
  caps against VOUT with a direct GND return to U3 GND/EP.
- NFC corner: GND tucks under U8 to a via, AC0/AC1 run in parallel
  lanes to C22 and the coil terminals (no crossing inside the ring).
- I2C moved from PB6/PB7 to PA9/PA10 (both I2C1); schematic and pin
  table updated, ERC clean.
- Docs: stackup, price, J2/FPC geometry, assembly order, front-parts
  height zone. Renders updated.

Co-Authored-By: Claude Opus 5.5 (1M context) <noreply@anthropic.com>
Connections:
- net SCL: now also U2.19 (PA9); no longer U2.25 (PB6)
- net SDA: now also U2.20 (PA10); no longer U2.26 (PB7)
Changed lines of the file:
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@@
 	(wire (pts (xy 124.46 101.6) (xy 121.92 101.6)) (stroke (width 0) (type default)))
 	(wire (pts (xy 124.46 104.14) (xy 121.92 104.14)) (stroke (width 0) (type default)))
-	(wire (pts (xy 124.46 109.22) (xy 121.92 109.22)) (stroke (width 0) (type default)))
-	(wire (pts (xy 124.46 111.76) (xy 121.92 111.76)) (stroke (width 0) (type default)))
+	(wire (pts (xy 154.94 106.68) (xy 157.48 106.68)) (stroke (width 0) (type default)))
+	(wire (pts (xy 154.94 109.22) (xy 157.48 109.22)) (stroke (width 0) (type default)))
 	(wire (pts (xy 58.42 91.44) (xy 58.42 88.9)) (stroke (width 0) (type default)))
 	(wire (pts (xy 58.42 111.76) (xy 58.42 114.3)) (stroke (width 0) (type default)))
@@
 	(hierarchical_label "NFC_VCC" (shape output) (at 121.92 101.6 180) (effects (font (size 1.27 1.27)) (justify right)))
 	(label "BTN2_N" (at 121.92 104.14 180) (effects (font (size 1.27 1.27)) (justify right bottom)))
-	(hierarchical_label "SCL" (shape output) (at 121.92 109.22 180) (effects (font (size 1.27 1.27)) (justify right)))
-	(hierarchical_label "SDA" (shape bidirectional) (at 121.92 111.76 180) (effects (font (size 1.27 1.27)) (justify right)))
+	(hierarchical_label "SCL" (shape output) (at 157.48 106.68 0) (effects (font (size 1.27 1.27)) (justify left)))
+	(hierarchical_label "SDA" (shape bidirectional) (at 157.48 109.22 0) (effects (font (size 1.27 1.27)) (justify left)))
 	(label "VBAT" (at 58.42 88.9 90) (effects (font (size 1.27 1.27)) (justify left bottom)))
 	(label "NRST" (at 71.12 96.52 0) (effects (font (size 1.27 1.27)) (justify left bottom)))
@@
 	(no_connect (at 124.46 96.52))
 	(no_connect (at 124.46 106.68))
-	(no_connect (at 154.94 106.68))
-	(no_connect (at 154.94 109.22))
+	(no_connect (at 124.46 109.22))
+	(no_connect (at 124.46 111.76))
 	(no_connect (at 154.94 116.84))
 	(no_connect (at 68.58 106.68))
